File: Home Automation with ESP32.kicad_sch (KiCad schematic)
At the start: 22 parts, among them J1 Conn_01x04_Pin, J1 PR13-5V-450-1C, J2 Screw_Terminal_01x04, J3 Screw_Terminal_01x03, K1 RAYEX-L90AS, Q1 S8050, Q2 S8050, SW1 SW_Push, SW2 SW_Push, U1 ESP32-WROOM-32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

Commit message: Relay-1 Completed in Schematic
Parts:
- added R2, R4: 1K, symbol Device:R
- R1: value R -> 1K
- R3: renamed from R2; value R -> 1K
Other:
- moved on the sheet: J1, Q2, U3
Changed lines of the file:
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@@
 	(symbol
 		(lib_id "Transistor_BJT:S8050")
-		(at 210.82 121.92 0)
-		(unit 1)
-		(exclude_from_sim no)
-		(in_bom yes)
-		(on_board yes)
-		(dnp no)
-		(fields_autoplaced yes)
+		(at 76.2 142.24 180)
+		(unit 1)
+		(exclude_from_sim no)
+		(in_bom yes)
+		(on_board yes)
+		(dnp no)
 		(property "Reference" "Q2"
-			(at 215.9 120.6499 0)
+			(at 71.12 143.5101 0)
 			(effects
 				(font
@@
 		)
 		(property "Value" "S8050"
-			(at 215.9 123.1899 0)
+			(at 71.12 140.9701 0)
 			(effects
 				(font
@@
 		)
 		(property "Footprint" "Package_TO_SOT_THT:TO-92_Inline"
-			(at 215.9 123.825 0)
+			(at 71.12 140.335 0)
 			(effects
 				(font
@@
 		)
 		(property "Datasheet" "http://www.unisonic.com.tw/datasheet/S8050.pdf"
-			(at 210.82 121.92 0)
+			(at 76.2 142.24 0)
 			(effects
 				(font
@@
 		)
 		(property "Description" "0.7A Ic, 20V Vce, Low Voltage High Current NPN Transistor, TO-92"
-			(at 210.82 121.92 0)
+			(at 76.2 142.24 0)
 			(effects
 				(font
@@
 		(on_board yes)
 		(dnp no)
-		(property "Reference" "R2"
+		(property "Reference" "R3"
 			(at 85.09 86.868 90)
 			(effects
@@
 			)
 		)
-		(property "Value" "R"
+		(property "Value" "1K"
 			(at 85.09 88.9 90)
 			(effects
@@
 			(project "Home Automation with ESP32"
 				(path "/7438dd54-9f08-4599-aef6-4a86e3e5147b"
-					(reference "R2")
+					(reference "R3")
 					(unit 1)
 				)
@@
 	(symbol
 		(lib_id "Isolator:PC817")
-		(at 209.55 59.69 0)
-		(unit 1)
-		(exclude_from_sim no)
-		(in_bom yes)
-		(on_board yes)
-		(dnp no)
-		(fields_autoplaced yes)
+		(at 107.95 144.78 180)
+		(unit 1)
+		(exclude_from_sim no)
+		(in_bom yes)
+		(on_board yes)
+		(dnp no)
 		(property "Reference" "U3"
-			(at 209.55 50.8 0)
+			(at 107.95 153.67 0)
 			(effects
 				(font
@@
 		)
 		(property "Value" "PC817"
-			(at 209.55 53.34 0)
+			(at 107.95 151.13 0)
 			(effects
 				(font
@@
 		)
 		(property "Footprint" "Package_DIP:DIP-4_W7.62mm"
-			(at 204.47 64.77 0)
+			(at 113.03 139.7 0)
 			(effects
 				(font
@@
 		)
 		(property "Datasheet" "http://www.soselectronic.cz/a_info/resource/d/pc817.pdf"
-			(at 209.55 59.69 0)
+			(at 107.95 144.78 0)
 			(effects
 				(font
@@
 		)
 		(property "Description" "DC Optocoupler, Vce 35V, CTR 50-300%, DIP-4"
-			(at 209.55 59.69 0)
+			(at 107.95 144.78 0)
 			(effects
 				(font
@@
 	)
 	(symbol
+		(lib_id "Device:R")
+		(at 123.19 147.32 90)
+		(unit 1)
+		(exclude_from_sim no)
+		(in_bom yes)
+		(on_board yes)
+		(dnp no)
+		(property "Reference" "R2"
+			(at 123.19 145.288 90)
+			(effects
+				(font
+					(size 1.27 1.27)
+				)
+			)
+		)
+		(property "Value" "1K"
+			(at 123.19 147.32 90)
+			(effects
+				(font
+					(size 1.27 1.27)
+				)
+			)
+		)
+		(property "Footprint" ""
+			(at 123.19 149.098 90)
+			(effects
+				(font
+					(size 1.27 1.27)
+				)
+				(hide yes)
+			)
+		)
+		(property "Datasheet" "~"
+			(at 123.19 147.32 0)
+			(effects
+				(font
+					(size 1.27 1.27)
+				)
+				(hide yes)
+			)
+		)
+		(property "Description" "Resistor"
+			(at 123.19 147.32 0)
+			(effects
+				(font
+					(size 1.27 1.27)
+				)
+				(hide yes)
+			)
+		)
+		(pin "2"
+		)
+		(pin "1"
+		)
+		(instances
+			(project "Home Automation with ESP32"
+				(path "/7438dd54-9f08-4599-aef6-4a86e3e5147b"
+					(reference "R2")
+					(unit 1)
+				)
+			)
+		)
+	)
+	(symbol
 		(lib_id "PR13-5V-450-1C:PR13-5V-450-1C")
-		(at 34.29 138.43 0)
-		(unit 1)
-		(exclude_from_sim no)
-		(in_bom yes)
-		(on_board yes)
-		(dnp no)
-		(fields_autoplaced yes)
+		(at 35.56 151.13 0)
+		(unit 1)
+		(exclude_from_sim no)
+		(in_bom yes)
+		(on_board yes)
+		(dnp no)
 		(property "Reference" "J1"
-			(at 50.8 130.81 0)
+			(at 51.562 160.02 0)
 			(effects
 				(font
@@
 		)
 		(property "Value" "PR13-5V-450-1C"
-			(at 50.8 133.35 0)
+			(at 52.07 162.306 0)
 			(effects
 				(font
@@
 		)
 		(property "Footprint" "PR135V4501C"
-			(at 63.5 233.35 0)
+			(at 64.77 246.05 0)
 			(effects
 				(font
@@
 		)
 		(property "Datasheet" "https://www.sameskydevices.com/product/resource/pr13.pdf"
-			(at 63.5 333.35 0)
+			(at 64.77 346.05 0)
 			(effects
 				(font
@@
 		)
 		(property "Description" "19 x 15.5 x 15.8 mm, 5 V, 10 A, SPDT (1 Form C), Power Relay"
-			(at 34.29 138.43 0)
+			(at 35.56 151.13 0)
 			(effects
 				(font
@@
 		)
 		(property "Height" "16.1"
-			(at 63.5 533.35 0)
+			(at 64.77 546.05 0)
 			(effects
 				(font
@@
 		)
 		(property "Manufacturer_Name" "Same Sky"
-			(at 63.5 633.35 0)
+			(at 64.77 646.05 0)
 			(effects
 				(font
@@
 		)
 		(property "Manufacturer_Part_Number" "PR13-5V-450-1C"
-			(at 63.5 733.35 0)
+			(at 64.77 746.05 0)
 			(effects
 				(font
@@
 		)
 		(property "Mouser Part Number" "179-PR13-5V-450-1C"
-			(at 63.5 833.35 0)
+			(at 64.77 846.05 0)
 			(effects
 				(font
@@
 		)
 		(property "Mouser Price/Stock" "https://www.mouser.co.uk/ProductDetail/CUI-Devices/PR13-5V-450-1C?qs=T%252BzbugeAwjjEdhOl%2F9q49A%3D%3D"
-			(at 63.5 933.35 0)
+			(at 64.77 946.05 0)
 			(effects
 				(font
@@
 		)
 		(property "Arrow Part Number" "PR13-5V-450-1C"
-			(at 63.5 1033.35 0)
+			(at 64.77 1046.05 0)
 			(effects
 				(font
@@
 		)
 		(property "Arrow Price/Stock" "https://www.arrow.com/en/products/pr13-5v-450-1c/cui-devices?region=nac"
-			(at 63.5 1133.35 0)
+			(at 64.77 1146.05 0)
 			(effects
 				(font
@@
 	(symbol
 		(lib_id "Device:R")
+		(at 88.9 142.24 90)
+		(unit 1)
+		(exclude_from_sim no)
+		(in_bom yes)
+		(on_board yes)
+		(dnp no)
+		(property "Reference" "R4"
+			(at 88.9 140.208 90)
+			(effects
+				(font
+					(size 1.27 1.27)
+				)
+			)
+		)
+		(property "Value" "1K"
+			(at 88.9 142.24 90)
+			(effects
+				(font
+					(size 1.27 1.27)
+				)
+			)
+		)
+		(property "Footprint" ""
+			(at 88.9 144.018 90)
+			(effects
+				(font
+					(size 1.27 1.27)
+				)
+				(hide yes)
+			)
+		)
+		(property "Datasheet" "~"
+			(at 88.9 142.24 0)
+			(effects
+				(font
+					(size 1.27 1.27)
+				)
+				(hide yes)
+			)
+		)
+		(property "Description" "Resistor"
+			(at 88.9 142.24 0)
+			(effects
+				(font
+					(size 1.27 1.27)
+				)
+				(hide yes)
+			)
+		)
+		(pin "2"
+		)
+		(pin "1"
+		)
+		(instances
+			(project "Home Automation with ESP32"
+				(path "/7438dd54-9f08-4599-aef6-4a86e3e5147b"
+					(reference "R4")
+					(unit 1)
+				)
+			)
+		)
+	)
+	(symbol
+		(lib_id "Device:R")
 		(at 118.11 93.98 90)
 		(unit 1)
@@
 			)
 		)
-		(property "Value" "R"
+		(property "Value" "1K"
 			(at 118.11 93.98 90)
 			(effects
